File: resources/KiCad/vpc-32-v1.kicad_pcb (KiCad board)
At the start: 2 copper layers, 0 parts

Commit message: modification au schéma électronique
Parts:
- added RCA-JACK: VAL**, RCA-JACK, F.Cu at (151.6, 84.1)
- added RCA-JACK: VAL**, RCA-JACK, F.Cu at (151.4, 104.6)
- added RJ-11: VAL**, RJ-11, F.Cu at (156.0, 126.0)
- added SDCard-Socket: VAL**, SDCard-Socket, F.Cu at (179.8, 172.5)
- added miniDIN-6: VAL**, miniDIN-6, F.Cu at (155.4, 146.6)
Routing:
- net (no net): track 0.00 -> 78.6 mm
Changed lines of the file:
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@@
     (thickness 1.6)
     (drawings 0)
-    (tracks 0)
+    (tracks 14)
     (zones 0)
-    (modules 0)
+    (modules 5)
     (nets 1)
   )
@@
     (mod_text_size 1 1)
     (mod_text_width 0.15)
-    (pad_size 1.524 1.524)
+    (pad_size 1.27 1.27)
     (pad_drill 0.6)
     (pad_to_mask_clearance 0)
     (aux_axis_origin 0 0)
-    (visible_elements FFFFF3BF)
+    (visible_elements 7FFFFFFF)
     (pcbplotparams
       (layerselection 3178497)
@@
     (add_net "")
   )
+  (module RCA-JACK (layer Dessus.Cu)
+    (at 151.638 84.074)
+    (fp_text reference RCA-JACK (at 0.1 -3.9) (layer Dessus.SilkS)
+      (effects (font (size 1 1) (thickness 0.15)))
+    )
+    (fp_text value VAL** (at 0 4.3) (layer Dessus.SilkS)
+      (effects (font (size 1 1) (thickness 0.15)))
+    )
+    (pad gnd1 smd rect (at 0 0) (size 1 1.6)
+      (layers Dessus.Cu Dessus.Pate Dessus.Masque)
+    )
+    (pad 1 smd rect (at 6.9 0) (size 2.2 2.6)
+      (layers Dessus.Cu Dessus.Pate Dessus.Masque)
+    )
+    (pad gnd2 smd rect (at 6.7 -6.35) (size 2.2 2.5)
+      (layers Dessus.Cu Dessus.Pate Dessus.Masque)
+    )
+    (pad gnd3 smd rect (at 6.7 6.35) (size 2.2 2.5)
+      (layers Dessus.Cu Dessus.Pate Dessus.Masque)
+    )
+  )
+  (module RCA-JACK (layer Dessus.Cu)
+    (at 151.384 104.648)
+    (fp_text reference RCA-JACK (at 0.1 -3.9) (layer Dessus.SilkS)
+      (effects (font (size 1 1) (thickness 0.15)))
+    )
+    (fp_text value VAL** (at 0 4.3) (layer Dessus.SilkS)
+      (effects (font (size 1 1) (thickness 0.15)))
+    )
+    (pad gnd1 smd rect (at 0 0) (size 1 1.6)
+      (layers Dessus.Cu Dessus.Pate Dessus.Masque)
+    )
+    (pad 1 smd rect (at 6.9 0) (size 2.2 2.6)
+      (layers Dessus.Cu Dessus.Pate Dessus.Masque)
+    )
+    (pad gnd2 smd rect (at 6.7 -6.35) (size 2.2 2.5)
+      (layers Dessus.Cu Dessus.Pate Dessus.Masque)
+    )
+    (pad gnd3 smd rect (at 6.7 6.35) (size 2.2 2.5)
+      (layers Dessus.Cu Dessus.Pate Dessus.Masque)
+    )
+  )
+  (module SDCard-Socket (layer Dessus.Cu)
+    (at 179.832 172.466 180)
+    (fp_text reference SDCard-Socket (at 16.6 -4.45 180) (layer Dessus.SilkS)
+      (effects (font (size 1 1) (thickness 0.15)))
+    )
+    (fp_text value VAL** (at 17.3 -1.15 180) (layer Dessus.SilkS)
+      (effects (font (size 1 1) (thickness 0.15)))
+    )
+    (pad 4 smd rect (at 1.5748 0.625 180) (size 2.54 1)
+      (layers Dessus.Cu Dessus.Pate Dessus.Masque)
+    )
+    (pad 3 smd rect (at 1.5748 -1.875 180) (size 2.5 1)
+      (layers Dessus.Cu Dessus.Pate Dessus.Masque)
+    )
+    (pad 2 smd rect (at 1.524 -4.375 180) (size 2.5 1)
+      (layers Dessus.Cu Dessus.Pate Dessus.Masque)
+    )
+    (pad 1 smd rect (at 1.5748 -6.875 180) (size 2.5 1)
+      (layers Dessus.Cu Dessus.Pate Dessus.Masque)
+    )
+    (pad 9 smd rect (at 1.5748 -9.375 180) (size 2.5 1)
+      (layers Dessus.Cu Dessus.Pate Dessus.Masque)
+    )
+    (pad 5 smd rect (at 1.6256 3.125 180) (size 2.54 1)
+      (layers Dessus.Cu Dessus.Pate Dessus.Masque)
+    )
+    (pad 6 smd rect (at 1.65 5.625 180) (size 2.54 1)
+      (layers Dessus.Cu Dessus.Pate Dessus.Masque)
+    )
+    (pad 7 smd rect (at 1.65 8.055 180) (size 2.54 1)
+      (layers Dessus.Cu Dessus.Pate Dessus.Masque)
+    )
+    (pad 8 smd rect (at 1.65 9.755 180) (size 2.54 1)
+      (layers Dessus.Cu Dessus.Pate Dessus.Masque)
+    )
+    (pad 10 smd rect (at 1.65 11.055 180) (size 2.54 0.7)
+      (layers Dessus.Cu Dessus.Pate Dessus.Masque)
+    )
+    (pad 11 smd rect (at 1.65 12.255 180) (size 2.54 0.7)
+      (layers Dessus.Cu Dessus.Pate Dessus.Masque)
+    )
+    (pad gnd smd rect (at 4.4 -11.565 180) (size 2.54 1.27)
+      (layers Dessus.Cu Dessus.Pate Dessus.Masque)
+    )
+    (pad gnd smd rect (at 4.85 13.765 180) (size 2.54 1.27)
+      (layers Dessus.Cu Dessus.Pate Dessus.Masque)
+    )
+    (pad gnd smd rect (at 27.43 -13.765 180) (size 2.54 1.27)
+      (layers Dessus.Cu Dessus.Pate Dessus.Masque)
+    )
+    (pad gnd smd rect (at 27.43 13.765 180) (size 2.54 1.26)
+      (layers Dessus.Cu Dessus.Pate Dessus.Masque)
+    )
+  )
+  (module RJ-11 (layer Dessus.Cu)
+    (at 155.956 125.984)
+    (fp_text reference RJ-11 (at 0 -5.4) (layer Dessus.SilkS)
+      (effects (font (size 1 1) (thickness 0.15)))
+    )
+    (fp_text value VAL** (at 0.2 5.4) (layer Dessus.SilkS)
+      (effects (font (size 1 1) (thickness 0.15)))
+    )
+    (fp_circle (center 0 -5.08) (end 3.048 -4.826) (layer Dessus.SilkS) (width 0.15))
+    (fp_circle (center 0 5.08) (end 3.302 5.08) (layer Dessus.SilkS) (width 0.15))
+    (fp_circle (center 0 5.08) (end 3.302 5.08) (layer Dessus.SilkS) (width 0.15))
+    (pad 1 thru_hole circle (at 6.35 2.54) (size 1.27 1.27) (drill 0.6)
+      (layers *.Cu *.Mask Dessus.SilkS)
+    )
+    (pad 2 thru_hole circle (at 8.89 1.27) (size 1.27 1.27) (drill 0.6)
+      (layers *.Cu *.Mask Dessus.SilkS)
+    )
+    (pad 3 thru_hole circle (at 6.35 -0.254) (size 1.27 1.27) (drill 0.6)
+      (layers *.Cu *.Mask Dessus.SilkS)
+    )
+    (pad 4 thru_hole circle (at 8.89 -1.778) (size 1.27 1.27) (drill 0.6)
+      (layers *.Cu *.Mask Dessus.SilkS)
+    )
+    (pad 5 thru_hole circle (at 6.35 -2.794) (size 1.27 1.27) (drill 0.6)
+      (layers *.Cu *.Mask Dessus.SilkS)
+    )
+    (pad 6 thru_hole circle (at 9.144 -4.572) (size 1.27 1.27) (drill 0.6)
+      (layers *.Cu *.Mask Dessus.SilkS)
+    )
+  )
+  (module miniDIN-6 (layer Dessus.Cu)
+    (at 155.448 146.558)
+    (fp_text reference miniDIN-6 (at -1.9 -3.4) (layer Dessus.SilkS)
+      (effects (font (size 1 1) (thickness 0.15)))
+    )
+    (fp_text value VAL** (at -0.4 3.2) (layer Dessus.SilkS)
+      (effects (font (size 1 1) (thickness 0.15)))
+    )
+    (fp_line (start -4.6736 -0.762) (end -4.6736 0.6604) (layer Dessus.SilkS) (width 0.15))
+    (fp_circle (center 0.8128 5.7404) (end 1.9812 5.842) (layer Dessus.SilkS) (width 0.15))
+    (fp_circle (center 0.8128 -5.7404) (end 1.9812 -5.6896) (layer Dessus.SilkS) (width 0.15))
+    (fp_circle (center 0 0) (end -1.143 0.127) (layer Dessus.SilkS) (width 0.15))
+    (pad 2 thru_hole circle (at 3.81 1.2954) (size 1.27 1.27) (drill 0.6)
+      (layers *.Cu *.Mask Dessus.SilkS)
+    )
+    (pad 1 thru_hole circle (at 3.81 -1.2954) (size 1.27 1.27) (drill 0.6)
+      (layers *.Cu *.Mask Dessus.SilkS)
+    )
+    (pad 4 thru_hole circle (at 3.81 3.3528) (size 1.27 1.27) (drill 0.6)
+      (layers *.Cu *.Mask Dessus.SilkS)
+    )
+    (pad 3 thru_hole circle (at 3.81 -3.3528) (size 1.27 1.27) (drill 0.6)
+      (layers *.Cu *.Mask Dessus.SilkS)
+    )
+    (pad 6 thru_hole circle (at 6.5532 3.3528) (size 1.27 1.27) (drill 0.6)
+      (layers *.Cu *.Mask Dessus.SilkS)
+    )
+    (pad 5 thru_hole circle (at 6.5532 -3.3528) (size 1.27 1.27) (drill 0.6)
+      (layers *.Cu *.Mask Dessus.SilkS)
+    )
+  )
+  (segment (start 153.416 186.436) (end 172.212 186.436) (width 0.254) (layer Dessous.Cu) (net 0))
+  (segment (start 172.212 186.436) (end 174.752 183.896) (width 0.254) (layer Dessous.Cu) (net 0))
+  (segment (start 153.416 158.75) (end 174.752 158.75) (width 0.254) (layer Dessous.Cu) (net 0))
+  (segment (start 174.752 158.75) (end 173.99 158.75) (width 0.254) (layer Dessous.Cu) (net 0))
+  (segment (start 156.972 98.298) (end 156.972 99.314) (width 0.254) (layer Dessous.Cu) (net 0))
+  (segment (start 151.638 105.41) (end 157.226 110.998) (width 0.254) (layer Dessous.Cu) (net 0))
+  (segment (start 151.638 104.648) (end 151.638 105.41) (width 0.254) (layer Dessous.Cu) (net 0))
+  (segment (start 156.972 99.314) (end 151.638 104.648) (width 0.254) (layer Dessous.Cu) (net 0))
+  (segment (start 157.226 90.424) (end 157.226 89.662) (width 0.254) (layer Dessous.Cu) (net 0))
+  (segment (start 157.226 78.74) (end 157.226 77.724) (width 0.254) (layer Dessous.Cu) (net 0))
+  (segment (start 152.146 83.82) (end 152.146 84.074) (width 0.254) (layer Dessous.Cu) (net 0))
+  (segment (start 157.226 78.74) (end 152.146 83.82) (width 0.254) (layer Dessous.Cu) (net 0))
+  (segment (start 152.146 84.582) (end 152.146 84.074) (width 0.254) (layer Dessous.Cu) (net 0))
+  (segment (start 157.226 89.662) (end 152.146 84.582) (width 0.254) (layer Dessous.Cu) (net 0))
 )
