File: resources/KiCad/vpc-32-v2.sch (KiCad schematic (older format))
At the start: 62 parts, among them CON1 Power jack, J1 SD_SOCKET, J2 PS/2, J3 video out, J4 RJ11, J5 audio out, K1 jumper, P1 gamepad 2, P2 ICSP, P3 gempad 1, Q1 2N3906, Q2 2N3904, SW1 reset, SW2 Power, U1 LM3940-3.3, U2 PIC32MX170F256B, U3 23LC1024, X1 10Mhz

Commit message: resume work
Parts:
- C1, C10, C11, C12, C13, C14, C15, C2, C3, C4, C5, C6, C7, C8, C9: symbol C -> C-RESCUE-vpc-32-v2
- D2, D3: symbol LED -> LED-RESCUE-vpc-32-v2
- R1, R10, R11, R12, R13, R14, R15, R16, R17, R18, R19, R2, R20, R21, R3, R4, R5, R6, R7, R8, R9, R? (x2): symbol R -> R-RESCUE-vpc-32-v2
